Commit message: mimimal working version for mapping

File: catkin_ws/src/my_robot/urdf/my_robot.xacro (robot description, xacro)
@@ -122,5 +122,5 @@
         </material>
     </gazebo>
-    <link name="camera">
+    <link name="camera_link">
         <inertial>
             <mass value="0.1"/>
@@ -148,5 +148,5 @@
         </visual>
     </link>
-    <gazebo reference="camera">
+    <gazebo reference="camera_link">
         <material>
             Gazebo/Green
@@ -175,4 +175,6 @@
             </geometry>
         </visual>
+    </link>
+    <link name="camera_link_optical">
     </link>
     <!--Joints-->
@@ -200,5 +202,5 @@
     <joint type="fixed" name="camera_joint">
         <origin xyz="0.2 0 0" rpy="0 0 0"/>
-        <child link="camera"/>
+        <child link="camera_link"/>
         <parent link="chassis"/>
         <axis xyz="0 1 0" rpy="0 0 0"/>
@@ -210,3 +212,8 @@
         <axis xyz="0 1 0" rpy="0 0 0"/>
     </joint>
+    <joint name="camera_optical_joint" type="fixed">
+        <origin xyz="0 0 0" rpy="-1.5707 0 -1.5707"/>
+        <parent link="camera_link"/>
+        <child link="camera_link_optical"/>
+    </joint>
 </robot>
